File: pcb/Echinos/Echinos.kicad_sch (KiCad schematic)
At the start: 33 parts, among them J1 Conn_01x06_Socket, J2 Conn_01x06_Socket, J3 Conn_01x06_Socket, J5 SATA-7p, J6 USB_B_Micro, J7 Conn_01x04_Socket, SW1 Reset, U1 Helios, U7 SRV05-4

Commit message: [PCB] - Save last state with Helios MCU board.   - Fix LCSC part numbers (C11, F2)   - Fix pad numbering for SK6812 to match footprint and update PCB traces   - Use another LCSC part for LEDs that is available for economic assembly   - Remove jumpers from BOM (remove warning in JLCPCB)   - Add 180° rotation to FPCs (J1, J2, J3) to match selected part in JLCPCB manufacturing   - Add 180° rotation to LEDs to match selected part in JLCPCB manufacturing
Parts:
- F2: LCSC C66452 -> C69688
- J1, J2, J3: FT Rotation Offset (none) -> 180
- J6: footprint Echinos:USB_Micro-B_type5_Amphenol_Horizontal -> Echinos:USB_Micro-B_Amphenol_type5_micro23_Horizontal
- JP0, JP11, JP13, JP14, JP15, JP16: now left out of the parts list
Changed lines of the file:
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@@
 			)
 		)
+		(property "FT Rotation Offset" "180"
+			(at 102.87 193.04 0)
+			(effects
+				(font
+					(size 1.27 1.27)
+				)
+				(hide yes)
+			)
+		)
 		(pin "3"
 		)
@@
 			)
 		)
-		(property "LCSC" "C66452"
+		(property "LCSC" "C69688"
 			(at 34.29 85.09 0)
 			(effects
@@
 		(unit 1)
 		(exclude_from_sim no)
-		(in_bom yes)
+		(in_bom no)
 		(on_board yes)
 		(dnp no)
@@
 			)
 		)
+		(property "FT Rotation Offset" "180"
+			(at 102.87 228.6 0)
+			(effects
+				(font
+					(size 1.27 1.27)
+				)
+				(hide yes)
+			)
+		)
 		(pin "3"
 		)
@@
 		(unit 1)
 		(exclude_from_sim no)
-		(in_bom yes)
+		(in_bom no)
 		(on_board yes)
 		(dnp no)
@@
 		(unit 1)
 		(exclude_from_sim no)
-		(in_bom yes)
+		(in_bom no)
 		(on_board yes)
 		(dnp no)
@@
 		(unit 1)
 		(exclude_from_sim no)
-		(in_bom yes)
+		(in_bom no)
 		(on_board yes)
 		(dnp no)
@@
 			)
 		)
-		(property "Footprint" "Echinos:USB_Micro-B_type5_Amphenol_Horizontal"
+		(property "Footprint" "Echinos:USB_Micro-B_Amphenol_type5_micro23_Horizontal"
 			(at 128.27 50.8 0)
 			(effects
@@
 		(unit 1)
 		(exclude_from_sim no)
-		(in_bom yes)
+		(in_bom no)
 		(on_board yes)
 		(dnp no)
@@
 			)
 		)
+		(property "FT Rotation Offset" "180"
+			(at 104.14 269.24 0)
+			(effects
+				(font
+					(size 1.27 1.27)
+				)
+				(hide yes)
+			)
+		)
 		(pin "3"
 		)
@@
 		(unit 1)
 		(exclude_from_sim no)
-		(in_bom yes)
+		(in_bom no)
 		(on_board yes)
 		(dnp no)

Commit message: [PCB] - Save last state with Helios MCU board.   - Move helios PCB on the bottom side to avoid conflict while typing on the outer pinky key   - Improve helios PCB (both top and bottom) with PCB edge, orientation information, standardization of holes sizes
Parts:
- U1: footprint Echinos:Helios_AH_USBdn -> Echinos:Helios_AH_USBup
Changed lines of the file:
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@@
 			)
 		)
-		(property "Footprint" "Echinos:Helios_AH_USBdn"
+		(property "Footprint" "Echinos:Helios_AH_USBup"
 			(at 372.11 72.39 0)
 			(effects

Commit message: [PCB] - Save last state with Helios MCU board and on board USB-C.
Parts:
- added C3: 10u, Capacitor_SMD:C_0805_2012Metric, symbol Device:C
- added D3: B5817WS, Diode_SMD:D_SOD-323_HandSoldering, symbol Device:D_Schottky
- added F3: 500mA, Fuse:Fuse_1206_3216Metric, symbol Device:Polyfuse
- added FB1: 600R, Resistor_SMD:R_0805_2012Metric, symbol Device:FerriteBead_Small
- added J8: USB_C_Receptacle_USB2.0, Connector_USB:USB_C_Receptacle_GCT_USB4105-xx-A_16P_TopMnt_Horizontal, symbol Connector:USB_C_Receptacle_USB2.0
- added R7, R8: 5.1k, Resistor_SMD:R_0805_2012Metric, symbol Device:R
- added U2, U7: USBLC6-2P6, Package_TO_SOT_SMD:SOT-23-6, symbol Power_Protection:USBLC6-2SC6
- J5: now not fitted; now left out of the parts list
- U7_bis1: renamed from U7; now not fitted; now left out of the parts list
Connections:
- net GND: now also C3.2, FB1.2, J8.A1 (GND), J8.A12 (GND), J8.B1 (GND), J8.B12 (GND), R7.2, R8.2, U2.2 (GND), U7.2 (GND); no longer U7_bis1.2 (VN)
- net RX: now also U7.4 (I/O2); no longer J6.2 (D-), J7.3 (Pin_3), U7_bis1.4 (IO3), U7_bis1.6 (IO4)
- net TX: now also U7.6 (I/O1); no longer J6.3 (D+), J7.2 (Pin_2), U7_bis1.1 (IO1), U7_bis1.3 (IO2)
- net VBUS_split: now also U7.5 (VBUS); no longer U7_bis1.5 (VP)
- new net: J8.B5 (CC2), R7.1
- new net: C3.1, F3.1, J8.A4 (VBUS), J8.A9 (VBUS), J8.B4 (VBUS), J8.B9 (VBUS)
- new net: D3.2 (A), F3.2
- new net: J8.A5 (CC1), R8.1
- new net: FB1.1, J8.S1 (SHIELD)
- new net P_RX: J6.3 (D+), J7.2 (Pin_2), U7.3 (I/O2)
- new net P_TX: J6.2 (D-), J7.3 (Pin_3), U7.1 (I/O1)
- new net P_USB+: J8.A6 (D+), J8.B6 (D+), U2.1 (I/O1)
- new net P_USB-: J8.A7 (D-), J8.B7 (D-), U2.3 (I/O2)
- new net USB+: U2.6 (I/O1)
- new net USB-: U2.4 (I/O2)
- new net VBUS_safe: D3.1 (K), U2.5 (VBUS)
- no-connect marks 3 -> 5
Other:
- note added: "ESD protection (USB-C)"
- note added: "Filter ESD (100-500Mhz) Filter high frequency noise Impedance should be in 50-100Ω range at 100Mhz Impedance drop quickly when moving toward ferrite current rating --> I_Circuit ~= 0.2 x I_CR"
- note added: "Tells host that we need 500mA"
- note added: "USB Computer/keyboard communication"
- note added: "Voltage clamp Reverse voltage protection"
- moved on the sheet: F2, H1, H2, H3, H4, H5, H6, JP11, JP12, S2, S3, S4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

Commit message: [PCB] - Save last state with on board RP2040.
Parts:
- removed J5: SATA-7p, Echinos:SATA_1x07_P1.27mm_pads_SMD, symbol Echinos:SATA-7p
- added C1: 1µ, Capacitor_SMD:C_0603_1608Metric_Pad1.08x0.95mm_HandSolder, symbol Device:C
- added C2: 4.7µ, Capacitor_SMD:C_0603_1608Metric_Pad1.08x0.95mm_HandSolder, symbol Device:C
- added D1: LED, Diode_SMD:D_SOD-323_HandSoldering, symbol Device:LED
- added JP205: 3x3_LED_jumper, Echinos:SolderJumper_Open_0.8x1.2mm, symbol Jumper:SolderJumper_2_Open
- added R1: 10k, Resistor_SMD:R_0402_1005Metric_Pad0.72x0.64mm_HandSolder, symbol Device:R
- added R12: 5.1k, Resistor_SMD:R_0402_1005Metric_Pad0.72x0.64mm_HandSolder, symbol Device:R
- added R9: 1k, Resistor_SMD:R_0402_1005Metric_Pad0.72x0.64mm_HandSolder, symbol Device:R
- added U3: XC6210B332MR-G, Package_TO_SOT_SMD:SOT-23-5_HandSoldering, symbol Regulator_Linear:XC6210B332MR
- R7, R8: footprint Resistor_SMD:R_0805_2012Metric -> Resistor_SMD:R_0402_1005Metric_Pad0.72x0.64mm_HandSolder; LCSC C27834 -> C25905
- U1: now not fitted
Connections:
- net VBUS_safe is gone; now on net +5V: D3.1 (K), U2.5 (VBUS)
- net +3.3V: now also C2.1, JP205.1 (A), U3.5 (VOUT)
- net +5V: now also C1.1, U3.1 (VIN), U3.3 (CE)
- net GND: now also C1.2, C2.2, D1.1 (K), R1.1, U3.2 (GND)
- net P_USB+: now also U2.3 (I/O2); no longer U2.1 (I/O1)
- net P_USB-: now also U2.1 (I/O1); no longer U2.3 (I/O2)
- net USB+: now also U2.4 (I/O2); no longer U2.6 (I/O1)
- net USB-: now also U2.6 (I/O1); no longer U2.4 (I/O2)
- net VBUS: now also D3.2 (A), F3.2, R12.2
- net VBUS_RAW: now reaches C3.1, F3.1, J8.A4 (VBUS), J8.A9 (VBUS), J8.B4 (VBUS), J8.B9 (VBUS)
- new net: D1.2 (A), R9.1
- new net: JP205.2 (B), R9.2
- new net RP2040/GPIO19: R1.2, R12.1
- no-connect marks 5 -> 8
Other:
- added sheet RP2040 (RP2040.kicad_sch)
- note added: "Max Current Output = 700mA Max Voltage Input = 6V"
- note added: "On/Off indicator"
- note added: "Voltage regulation"
- moved on the sheet: C3, D3, F2, F3, J1, J2, J3, J6, J7, JP15, JP16, R15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

Commit message: [PCB] - Save last state with on board RP2040.
Parts:
- removed SW1: Reset, Button_Switch_SMD:SW_SPST_TL3342, symbol Switch:SW_Push
- removed U7_bis1: SRV05-4, Package_TO_SOT_SMD:SOT-23-6, symbol Power_Protection:SRV05-4
- added J10: TagConnect_6pins, Connector:Tag-Connect_TC2030-IDC-FP_2x03_P1.27mm_Vertical, symbol Connector:Conn_ARM_SWD_TagConnect_TC2030
- added J5: Conn_01x05_Socket, Connector_PinHeader_2.00mm:PinHeader_1x05_P2.00mm_Vertical, symbol Connector:Conn_01x05_Socket
- added J9: Conn_01x03_Socket, Connector_JST:JST_SH_BM03B-SRSS-TB_1x03-1MP_P1.00mm_Vertical, symbol Connector:Conn_01x03_Pin
- added R18, R19: 100, Resistor_SMD:R_0805_2012Metric, symbol Device:R
- added SW3, SW4: Reset, Button_Switch_SMD:SW_SPST_TS-1088-xR020, symbol Switch:SW_Push
- added U8: 74LVC1T45, Package_TO_SOT_SMD:SOT-563, symbol Logic_LevelTranslator:SN74LVC1T45DRL
- JP0, JP11: footprint Jumper:SolderJumper-2_P1.3mm_Bridged_Pad1.0x1.5mm -> Jumper:SolderJumper-2_P1.3mm_Bridged_RoundedPad1.0x1.5mm
- JP12: footprint Jumper:SolderJumper-3_P1.3mm_Bridged12_Pad1.0x1.5mm_NumberLabels -> Jumper:SolderJumper-3_P1.3mm_Bridged12_RoundedPad1.0x1.5mm_NumberLabels
- JP13, JP14, JP15, JP16: footprint Jumper:SolderJumper-2_P1.3mm_Open_Pad1.0x1.5mm -> Jumper:SolderJumper-2_P1.3mm_Open_RoundedPad1.0x1.5mm
- JP205: footprint Echinos:SolderJumper_Open_0.8x1.2mm -> Jumper:SolderJumper-2_P1.3mm_Bridged_RoundedPad1.0x1.5mm; symbol Jumper:SolderJumper_2_Open -> Jumper:SolderJumper_2_Bridged; now left out of the parts list
Connections:
- net +3.3V: now also J5.5 (Pin_5), U8.1 (VCCA), U8.5 (DIR)
- net +5V: now also U8.6 (VCCB)
- net GND: now also J5.1 (Pin_1), SW3.2, SW4.1, U8.2 (GND)
- net col1: now also J1.5 (Pin_5); no longer J1.2 (Pin_2)
- net col2: now also J1.4 (Pin_4); no longer J1.3 (Pin_3), J2.6 (Pin_6)
- net col3: now also J1.3 (Pin_3); no longer J1.4 (Pin_4)
- net col4: now also J1.2 (Pin_2); no longer J1.5 (Pin_5)
- net col5: now also J1.1 (Pin_1); no longer J1.6 (Pin_6)
- net reset: now also J5.4 (Pin_4), SW3.1, SW4.2
- net rgb: now also U8.3 (A); no longer JP11.1 (A)
- net row6: now also J1.6 (Pin_6); no longer J1.1 (Pin_1)
- new net col6: J2.6 (Pin_6)
- new net rgb_5V: JP11.1 (A), U8.4 (B)
- new net swclk: J5.2 (Pin_2)
- new net swdio: J5.3 (Pin_3)
- no-connect marks 8 -> 7
Other:
- sheet Matrix ports: added none; removed adx, ady
- sheet RP2040 ports: added SWCLK, SWDIO, USB+, USB-, ~{RST}; removed USB_D+, USB_D-
- note added: "Coplanar differential USB pairs (JLCPCB, 2 Layers JLC0216) - Dieletric=4.5 - H=1.4650 - eps=0.02 JLCPCB non coplanar (W=0.4862mm, S=0.15mm) JLCPCB coplanar (W=0.34mm, S=0.15mm) Altium coplanar (W=0.4086mm, S=0.127mm) Due to imperfect coplanar plane --> W = 0.381"
- note added: "Debug (Optional)"
- note added: "Header with all required pins to debug."
- note added: "Raspberry Pi Debug Probe"
- note added: "Universal tag connector"
- moved on the sheet: JP11, JP205
