File: pcb/Echinos/Echinos_Right.kicad_pcb (KiCad board)
At the start: 2 copper layers, 167.4 x 138.9 mm, 134 parts, among them J200 USB_B_Micro, J201 Conn_01x04_Socket, J202 Conn_01x12_Socket, J203 Conn_01x06_Socket, J204 Conn_01x06_Socket, J205 Conn_01x06_Socket, J206 USB_C_Receptacle_USB2.0, J207 Conn_01x05_Socket, SW200 SW_Push, SW201 SW_Push, SW202 SW_Push, SW203 SW_Push, SW204 SW_Push, SW205 SW_Push, SW206 SW_Push, SW207 SW_Push, SW208 SW_Push, SW209 SW_Push, SW210 SW_Push, SW211 SW_Push, SW212 SW_Push, SW213 SW_Push, SW214 SW_Push, SW215 SW_Push, SW216 SW_Push, SW217 SW_Push, SW218 SW_Push, SW219 SW_Push, SW220 SW_Push, SW221 SW_Push, SW222 SW_Push, SW223 SW_Push, SW224 Button, SW225 Button, SW226 Button, SW227 Button, U200 W25Q128JVP, U201 RP2040, U202 USBLC6-2P6, U203 74LVC1T45, U204 USBLC6-2P6, U205 XC6210B332MR-G, Y200 Crystal_GND24

Commit message: 💥 [PCB] - Split schematic for left and right halves.   - Required to create a common PCB to lower the manufacturing cost
Connections:
- net /Split/Backlight/backlight_in renamed /Right/Backlight/backlight_in
- net /Split/P_USB+ renamed /Right/P_USB+
- net /Split/P_USB- renamed /Right/P_USB-
- net /Split/RP2040/GPIO12 renamed /Right/RP2040/GPIO12
- net /Split/RP2040/GPIO18 renamed /Right/RP2040/GPIO18
- net /Split/RP2040/GPIO19 renamed /Right/RP2040/GPIO19
- net /Split/RP2040/QSPI_SCLK renamed /Right/RP2040/QSPI_SCLK
- net /Split/RP2040/QSPI_SD0 renamed /Right/RP2040/QSPI_SD0
- net /Split/RP2040/QSPI_SD1 renamed /Right/RP2040/QSPI_SD1
- net /Split/RP2040/QSPI_SD2 renamed /Right/RP2040/QSPI_SD2
- net /Split/RP2040/QSPI_SD3 renamed /Right/RP2040/QSPI_SD3
- net /Split/RP2040/QSPI_SS renamed /Right/RP2040/QSPI_SS
- net /Split/USB+ renamed /Right/USB+
- net /Split/USB- renamed /Right/USB-
